Commit message: urdf another files

File: urdf/common_propertes.xacro (robot description, xacro)
@@ -1 +1,9 @@
 <?xml version="1.0"?>
+<robot xmlns:xacro="http://www.ros.org/wiki/xacro">
+    <material name="blue">
+        <color rgba="0.6 0 0 1"/>
+    </material>
+    <material name="gray">
+        <color rgba="0.5 0.5 0.5 1"/>
+    </material>
+</robot>

File: urdf/mobile_base.xacro (robot description, xacro)
@@ -1 +1,93 @@
 <?xml version="1.0"?>
+<robot name="my_robot" xmlns:xacro="http://www.ros.org/wiki/xacro">
+    <!-- <xacro:include filename="common_propertes.xacro" /> -->
+    <xacro:property name="base_lenght" value="0.6"/>
+    <xacro:property name="base_width" value="0.4"/>
+    <xacro:property name="base_height" value="0.2"/>
+    <xacro:property name="wheel_radius" value="0.1"/>
+    <xacro:property name="wheel_lenght" value="0.05"/>
+    <!-- <xacro:macro name="example_macro" param="a b c">
+        <link name="dummy_link">
+            <visual>
+                <geometry>
+                    <box size="${a} ${b} ${c}" />
+                </geometry>
+            </visual>
+        </link>
+    </xacro:macro>
+    <xacro:example_macro a="2" b="3" c="4" /> -->
+    <link name="base_footpriint" />
+    <link name="base_link">
+        <visual>
+            <geometry>
+                <box size="${base_lenght} ${base_width} ${base_height}" />
+            </geometry>
+            <origin xyz="0 0 ${base_height / 2.0}" rpy="0 0 0" />
+            <material name="blue" />
+        </visual>
+    </link>
+    <!-- wheel -->
+    <xacro:macro name="wheel_link" params="prefix">
+        <link name="${prefix}_wheel_link">
+            <visual>
+                <geometry>
+                    <cylinder radius="${wheel_radius}" length="${wheel_lenght}" />
+                </geometry>
+                <origin xyz="0 0 0" rpy="${pi / 2} 0 0" />
+                <material name="gray" />
+            </visual>
+        </link>
+    </xacro:macro>
+    <link name="caster_wheel_link">
+        <visual>
+            <geometry>
+                <sphere radius="${wheel_radius / 2.0}"/>
+            </geometry>
+            <origin xyz="0 0 0" rpy="0 0 0" />
+            <material name="gray" />
+        </visual>
+    </link>
+    <xacro:wheel_link prefix="right" />
+    <xacro:wheel_link prefix="left" />
+    <!-- <link name="right_wheel_link">
+        <visual>
+            <geometry>
+                <cylinder radius="${wheel_radius}" length="${wheel_lenght}" />
+            </geometry>
+            <origin xyz="0 0 0" rpy="${pi / 2} 0 0" />
+            <material name="gray" />
+        </visual>
+    </link>
+    <link name="left_wheel_link">
+        <visual>
+            <geometry>
+                <cylinder radius="${wheel_radius}" length="${wheel_lenght}" />
+            </geometry>
+            <origin xyz="0 0 0" rpy="${pi / 2} 0 0" />
+            <material name="gray" />
+        </visual>
+    </link> -->
+    <!-- joint -->
+    <joint name="base_joint" type="fixed">
+        <parent link="base_footpriint" />
+        <child link="base_link" />
+        <origin xyz="0 0 ${wheel_radius}" rpy="0 0 0" />
+    </joint>
+    <joint name="base_right_wheel_joint" type="continuous">
+        <parent link="base_link" />
+        <child link="right_wheel_link" />
+        <origin xyz="${-base_lenght / 4.0} ${-(base_width + wheel_lenght) / 2.0} 0" rpy="0 0 0" />
+        <axis xyz="0 1 0" />
+    </joint>
+    <joint name="base_left_wheel_joint" type="continuous">
+        <parent link="base_link" />
+        <child link="left_wheel_link" />
+        <origin xyz="${-base_lenght / 4.0} ${(base_width + wheel_lenght) / 2.0} 0" rpy="0 0 0" />
+        <axis xyz="0 1 0" />
+    </joint>
+    <joint name="base_caster_wheel_joint" type="fixed">
+        <parent link="base_link" />
+        <child link="caster_wheel_link" />
+        <origin xyz="${base_lenght / 3.0} 0 ${-wheel_radius / 2.0}" rpy="0 0 0" />
+    </joint>
+</robot>

File: urdf/my_robot.urdf.xacro (robot description, xacro)
@@ -1,98 +1,5 @@
 <?xml version="1.0"?>
 <robot name="my_robot" xmlns:xacro="http://www.ros.org/wiki/xacro">
-    <xacro:property name="base_lenght" value="0.6"/>
-    <xacro:property name="base_width" value="0.4"/>
-    <xacro:property name="base_height" value="0.2"/>
-    <xacro:property name="wheel_radius" value="0.1"/>
-    <xacro:property name="wheel_lenght" value="0.05"/>
-    <!-- <xacro:macro name="example_macro" param="a b c">
-        <link name="dummy_link">
-            <visual>
-                <geometry>
-                    <box size="${a} ${b} ${c}" />
-                </geometry>
-            </visual>
-        </link>
-    </xacro:macro>
-    <xacro:example_macro a="2" b="3" c="4" /> -->
-    <material name="blue">
-        <color rgba="0.9 0 0 1"/>
-    </material>
-    <material name="gray">
-        <color rgba="0.5 0.5 0.5 1"/>
-    </material>
-    <link name="base_footpriint" />
-    <link name="base_link">
-        <visual>
-            <geometry>
-                <box size="${base_lenght} ${base_width} ${base_height}" />
-            </geometry>
-            <origin xyz="0 0 ${base_height / 2.0}" rpy="0 0 0" />
-            <material name="blue" />
-        </visual>
-    </link>
-    <!-- wheel -->
-    <xacro:macro name="wheel_link" params="prefix">
-        <link name="${prefix}_wheel_link">
-            <visual>
-                <geometry>
-                    <cylinder radius="${wheel_radius}" length="${wheel_lenght}" />
-                </geometry>
-                <origin xyz="0 0 0" rpy="${pi / 2} 0 0" />
-                <material name="gray" />
-            </visual>
-        </link>
-    </xacro:macro>
-    <link name="caster_wheel_link">
-        <visual>
-            <geometry>
-                <sphere radius="${wheel_radius / 2.0}"/>
-            </geometry>
-            <origin xyz="0 0 0" rpy="0 0 0" />
-            <material name="gray" />
-        </visual>
-    </link>
-    <xacro:wheel_link prefix="right" />
-    <xacro:wheel_link prefix="left" />
-    <!-- <link name="right_wheel_link">
-        <visual>
-            <geometry>
-                <cylinder radius="${wheel_radius}" length="${wheel_lenght}" />
-            </geometry>
-            <origin xyz="0 0 0" rpy="${pi / 2} 0 0" />
-            <material name="gray" />
-        </visual>
-    </link>
-    <link name="left_wheel_link">
-        <visual>
-            <geometry>
-                <cylinder radius="${wheel_radius}" length="${wheel_lenght}" />
-            </geometry>
-            <origin xyz="0 0 0" rpy="${pi / 2} 0 0" />
-            <material name="gray" />
-        </visual>
-    </link> -->
-    <!-- joint -->
-    <joint name="base_joint" type="fixed">
-        <parent link="base_footpriint" />
-        <child link="base_link" />
-        <origin xyz="0 0 ${wheel_radius}" rpy="0 0 0" />
-    </joint>
-    <joint name="base_right_wheel_joint" type="continuous">
-        <parent link="base_link" />
-        <child link="right_wheel_link" />
-        <origin xyz="${-base_lenght / 4.0} ${-(base_width + wheel_lenght) / 2.0} 0" rpy="0 0 0" />
-        <axis xyz="0 1 0" />
-    </joint>
-    <joint name="base_left_wheel_joint" type="continuous">
-        <parent link="base_link" />
-        <child link="left_wheel_link" />
-        <origin xyz="${-base_lenght / 4.0} ${(base_width + wheel_lenght) / 2.0} 0" rpy="0 0 0" />
-        <axis xyz="0 1 0" />
-    </joint>
-    <joint name="base_caster_wheel_joint" type="fixed">
-        <parent link="base_link" />
-        <child link="caster_wheel_link" />
-        <origin xyz="${base_lenght / 3.0} 0 ${-wheel_radius / 2.0}" rpy="0 0 0" />
-    </joint>
+    <xacro:include filename="common_propertes.xacro" />
+    <xacro:include filename="mobile_base.xacro" />
 </robot>

Commit message: urdf collision

File: urdf/common_propertes.xacro (robot description, xacro)
@@ -7,3 +7,30 @@
         <color rgba="0.5 0.5 0.5 1"/>
     </material>
+    <xacro:macro name="box_inertia" params="m l w h xyz rpy">
+        <inertial>
+            <origin xyz="${xyz}" rpy="${rpy}" />
+            <mass value="${m}" />
+            <inertia ixx="${(m/12) * (h*h + l*l)}" ixy="0" ixz="0"
+                     iyy="${(m/12) * (w*w + l*l)}" iyz="0"
+                     izz="${(m/12) * (w*w + h*h)}" />
+        </inertial>
+    </xacro:macro>
+    <xacro:macro name="cylinder_inertia" params="m r h xyz rpy">
+        <inertial>
+            <origin xyz="${xyz}" rpy="${rpy}" />
+            <mass value="${m}" />
+            <inertia ixx="${(m/12) * (3*r*r + h*h)}" ixy="0" ixz="0"
+                     iyy="${(m/12) * (3*r*r + h*h)}" iyz="0"
+                     izz="${(m/2) * (r*r)}" />
+        </inertial>
+    </xacro:macro>
+    <xacro:macro name="sphere_inertia" params="m r xyz rpy">
+        <inertial>
+            <origin xyz="${xyz}" rpy="${rpy}" />
+            <mass value="${m}" />
+            <inertia ixx="${((2/5) * m) * (r*r)}" ixy="0" ixz="0"
+                     iyy="${((2/5) * m) * (r*r)}" iyz="0"
+                     izz="${((2/5) * m) * (r*r)}" />
+        </inertial>
+    </xacro:macro>
 </robot>

File: urdf/mobile_base.xacro (robot description, xacro)
@@ -26,4 +26,12 @@
             <material name="blue" />
         </visual>
+        <collision>
+            <geometry>
+                <box size="${base_lenght} ${base_width} ${base_height}" />
+            </geometry>
+            <origin xyz="0 0 ${base_height / 2.0}" rpy="0 0 0" />
+        </collision>
+        <xacro:box_inertia m="5.0" l="${base_lenght}" w="${base_width}" h="${base_height}"
+                           xyz="0 0 ${base_height / 2.0}" rpy="0 0 0" />
     </link>
     <!-- wheel -->
@@ -37,4 +45,12 @@
                 <material name="gray" />
             </visual>
+            <collision>
+                <geometry>
+                    <cylinder radius="${wheel_radius}" length="${wheel_lenght}" />
+                </geometry>
+                <origin xyz="0 0 0" rpy="${pi / 2} 0 0" />
+            </collision>
+            <xacro:cylinder_inertia m="1.0" r="${wheel_radius}" h="${wheel_lenght}"
+                                    xyz="0 0 0" rpy="${pi / 2} 0 0" />
         </link>
     </xacro:macro>
@@ -47,4 +63,11 @@
             <material name="gray" />
         </visual>
+        <collision>
+            <geometry>
+                <sphere radius="${wheel_radius / 2.0}"/>
+            </geometry>
+        </collision>
+        <xacro:sphere_inertia m="5.0" r="${wheel_radius / 2.0}"
+                              xyz="0 0 0" rpy="0 0 0" />
     </link>
     <xacro:wheel_link prefix="right" />
